Commit message: feat(test): add random GPU test and URDF backups

File: xarm7 copy 2.urdf (robot description, URDF)
Before this commit: robot UF_ROBOT, 18 links, 17 joints
Links:
- link left_finger: geometry visual mesh filename=package://xarm_description/meshes/gripper/xarm/left_finger.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
- link left_outer_knuckle: geometry visual mesh filename=package://xarm_description/meshes/gripper/xarm/left_outer_k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
- link right_finger: geometry visual mesh filename=package://xarm_description/meshes/gripper/xarm/right_finger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
- link right_outer_knuckle: geometry visual mesh filename=package://xarm_description/meshes/gripper/xarm/right_outer_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
- link xarm_gripper_base_link: geometry visual mesh filename=package://xarm_description/meshes/gripper/xarm/base_link.stl

File: xarm7 copy.urdf (robot description, URDF)
Before this commit: robot UF_ROBOT, 18 links, 17 joints
Links:
- link left_finger: geometry visual mesh filename=package://xarm_description/meshes/gripper/xarm/left_finger.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
- link left_outer_knuckle: geometry visual mesh filename=package://xarm_description/meshes/gripper/xarm/left_outer_k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
- link right_finger: geometry visual mesh filename=package://xarm_description/meshes/gripper/xarm/right_finger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
- link right_outer_knuckle: geometry visual mesh filename=package://xarm_description/meshes/gripper/xarm/right_outer_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
- link xarm_gripper_base_link: geometry visual mesh filename=package://xarm_description/meshes/gripper/xarm/base_link.stl
