Commit message: tune(urdf): remove xArm7 gripper base visuals

File: xarm7.urdf (robot description, URDF)
Before this commit: robot UF_ROBOT, 18 links, 17 joints
Links:
- link xarm_gripper_base_link: geometry 

Commit message: tune(urdf): comment xArm7 gripper assembly

File: xarm7.urdf (robot description, URDF)
Before this commit: robot UF_ROBOT, 18 links, 17 joints
Links:
- removed link left_finger
- removed link left_inner_knuckle
- removed link left_outer_knuckle
- removed link link_tcp
- removed link right_finger
- removed link right_inner_knuckle
- removed link right_outer_knuckle
- removed link xarm_gripper_base_link
Joints:
- removed joint drive_joint
- removed joint gripper_fix
- removed joint joint_tcp
- removed joint left_finger_joint
- removed joint left_inner_knuckle_joint
- removed joint right_finger_joint
- removed joint right_inner_knuckle_joint
- removed joint right_outer_knuckle_joint

Commit message: tune(urdf): restore gripper links with hidden visuals

File: xarm7.urdf (robot description, URDF)
Before this commit: robot UF_ROBOT, 10 links, 9 joints
Links:
- added link left_finger, mass 0.048304
- added link left_inner_knuckle, mass 0.0230125781256706
- added link left_outer_knuckle, mass 0.033618
- added link link_tcp
- added link right_finger, mass 0.048304
- added link right_inner_knuckle, mass 0.023013
- added link right_outer_knuckle, mass 0.033618
- added link xarm_gripper_base_link, mass 0.54156
Joints:
- added joint drive_joint: type revolute, parent xarm_gripper_base_link, child left_outer_knuckle, origin xyz=0 0.035 0.059098 rpy=0 0 0, axis 1 0 0, limit lower=0 upper=0.85 effort=50 velocity=2
- added joint gripper_fix: type fixed, parent link_eef, child xarm_gripper_base_link, origin xyz=0 0 0 rpy=0 0 0
- added joint joint_tcp: type fixed, parent xarm_gripper_base_link, child link_tcp, origin xyz=0 0 0.172 rpy=0 0 0
- added joint left_finger_joint: type revolute, parent left_outer_knuckle, child left_finger, origin xyz=0 0.035465 0.042039 rpy=0 0 0, axis -1 0 0, limit lower=0 upper=0.85 effort=50 velocity=2, mimic joint=drive_joint multiplier=1 offset=0
- added joint left_inner_knuckle_joint: type revolute, parent xarm_gripper_base_link, child left_inner_knuckle, origin xyz=0 0.02 0.074098 rpy=0 0 0, axis 1 0 0, limit lower=0 upper=0.85 effort=50 velocity=2, mimic joint=drive_joint multiplier=1 offset=0
- added joint right_finger_joint: type revolute, parent right_outer_knuckle, child right_finger, origin xyz=0 -0.035465 0.042039 rpy=0 0 0, axis 1 0 0, limit lower=0 upper=0.85 effort=50 velocity=2, mimic joint=drive_joint multiplier=1 offset=0
- added joint right_inner_knuckle_joint: type revolute, parent xarm_gripper_base_link, child right_inner_knuckle, origin xyz=0 -0.02 0.074098 rpy=0 0 0, axis -1 0 0, limit lower=0 upper=0.85 effort=50 velocity=2, mimic joint=drive_joint multiplier=1 offset=0
- added joint right_outer_knuckle_joint: type revolute, parent xarm_gripper_base_link, child right_outer_knuckle, origin xyz=0 -0.035 0.059098 rpy=0 0 0, axis -1 0 0, limit lower=0 upper=0.85 effort=50 velocity=2, mimic joint=drive_joint multiplier=1 offset=0

Commit message: tune(urdf): disable xArm7 collision meshes

File: xarm7.urdf (robot description, URDF)
Before this commit: robot UF_ROBOT, 18 links, 17 joints
Links:
- link left_finger: geometry visual mesh filename=package://xarm_description/meshes/gripper/xarm/left_finger.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
- link left_inner_knuckle: geometry visual mesh filename=package://xarm_description/meshes/gripper/xarm/left_inner_k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
- link left_outer_knuckle: geometry visual mesh filename=package://xarm_description/meshes/gripper/xarm/left_outer_k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
- link link1: geometry visual mesh filename=package://xarm_description/meshes/xarm7/visual/link1.stl
- link link2: geometry visual mesh filename=package://xarm_description/meshes/xarm7/visual/link2.stl
- link link3: geometry visual mesh filename=package://xarm_description/meshes/xarm7/visual/link3.stl
- link link4: geometry visual mesh filename=package://xarm_description/meshes/xarm7/visual/link4.stl
- link link5: geometry visual mesh filename=package://xarm_description/meshes/xarm7/visual/link5.stl
- link link6: geometry visual mesh filename=package://xarm_description/meshes/xarm7/visual/link6.stl
- link link7: geometry visual mesh filename=package://xarm_description/meshes/xarm7/visual/link7.stl
- link right_finger: geometry visual mesh filename=package://xarm_description/meshes/gripper/xarm/right_finger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
- link right_inner_knuckle: geometry visual mesh filename=package://xarm_description/meshes/gripper/xarm/right_inner_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
- link right_outer_knuckle: geometry visual mesh filename=package://xarm_description/meshes/gripper/xarm/right_outer_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
- link xarm_gripper_base_link: geometry visual mesh filename=package://xarm_description/meshes/gripper/xarm/base_link.stl

Commit message: revert: restore full xArm7 URDF

File: xarm7.urdf (robot description, URDF)
Before this commit: robot UF_ROBOT, 18 links, 17 joints
Links:
- link left_finger: geometry collision mesh filename=package://xarm_description/meshes/gripper/xarm/left_finger.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; visual mesh filename=package://xarm_description/meshes/gripper/xarm/left_finger.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
- link left_inner_knuckle: geometry collision mesh filename=package://xarm_description/meshes/gripper/xarm/left_inner_k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; visual mesh filename=package://xarm_description/meshes/gripper/xarm/left_inner_k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
- link left_outer_knuckle: geometry collision mesh filename=package://xarm_description/meshes/gripper/xarm/left_outer_k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; visual mesh filename=package://xarm_description/meshes/gripper/xarm/left_outer_k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
- link link1: geometry collision mesh filename=package://xarm_description/meshes/xarm7/visual/link1.stl; visual mesh filename=package://xarm_description/meshes/xarm7/visual/link1.stl
- link link2: geometry collision mesh filename=package://xarm_description/meshes/xarm7/visual/link2.stl; visual mesh filename=package://xarm_description/meshes/xarm7/visual/link2.stl
- link link3: geometry collision mesh filename=package://xarm_description/meshes/xarm7/visual/link3.stl; visual mesh filename=package://xarm_description/meshes/xarm7/visual/link3.stl
- link link4: geometry collision mesh filename=package://xarm_description/meshes/xarm7/visual/link4.stl; visual mesh filename=package://xarm_description/meshes/xarm7/visual/link4.stl
- link link5: geometry collision mesh filename=package://xarm_description/meshes/xarm7/visual/link5.stl; visual mesh filename=package://xarm_description/meshes/xarm7/visual/link5.stl
- link link6: geometry collision mesh filename=package://xarm_description/meshes/xarm7/visual/link6.stl; visual mesh filename=package://xarm_description/meshes/xarm7/visual/link6.stl
- link link7: geometry collision mesh filename=package://xarm_description/meshes/end_tool/collision/end_to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; visual mesh filename=package://xarm_description/meshes/xarm7/visual/link7.stl
- link right_finger: geometry collision mesh filename=package://xarm_description/meshes/gripper/xarm/right_finger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; visual mesh filename=package://xarm_description/meshes/gripper/xarm/right_finger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
- link right_inner_knuckle: geometry collision mesh filename=package://xarm_description/meshes/gripper/xarm/right_inner_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; visual mesh filename=package://xarm_description/meshes/gripper/xarm/right_inner_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
- link right_outer_knuckle: geometry collision mesh filename=package://xarm_description/meshes/gripper/xarm/right_outer_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; visual mesh filename=package://xarm_description/meshes/gripper/xarm/right_outer_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
- link xarm_gripper_base_link: geometry collision mesh filename=package://xarm_description/meshes/gripper/xarm/base_link.stl; visual mesh filename=package://xarm_description/meshes/gripper/xarm/base_link.stl

Commit message: tune(urdf): adjust xArm7 joint limit

File: xarm7.urdf (robot description, URDF)
Before this commit: robot UF_ROBOT, 18 links, 17 joints
Joints:
- joint drive_joint: limit lower=0 upper=0.85 effort=50 velocity=2 -> lower=0.05 upper=0.84 effort=50 velocity=2

Commit message: refactor: archive legacy xarm7 MJCF experiments

File: xarm7.urdf (robot description, URDF)
Before this commit: robot UF_ROBOT, 18 links, 17 joints
Joints:
- joint drive_joint: limit lower=0.05 upper=0.84 effort=50 velocity=2 -> lower=0 upper=0.85 effort=50 velocity=2
