Commit message: feat: add xArm ball end-effector agent

File: xarm7_ball_ee.urdf (robot description, URDF)
Before this commit: robot UF_ROBOT, 18 links, 17 joints
Links:
- added link link_tcp_ball, mass 0.05; collision sphere radius=0.04; visual sphere radius=0.04
- link left_finger: geometry visual mesh filename=package://xarm_description/meshes/gripper/xarm/left_finger.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
- link right_finger: geometry visual mesh filename=package://xarm_description/meshes/gripper/xarm/right_finger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
- link right_outer_knuckle: geometry visual mesh filename=package://xarm_description/meshes/gripper/xarm/right_outer_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
Joints:
- added joint joint_tcp_ball: type fixed, parent link_tcp, child link_tcp_ball, origin xyz=0 0 0 rpy=0 0 0
