Commit message: feat: update xArm FT sensor URDF assets

File: xarm7_1305_realsense.urdf (robot description, URDF)
Before this commit: robot UF_ROBOT, 27 links, 26 joints
Links:
- added link link_tcp_ball, mass 0.05; collision sphere radius=0.04; visual sphere radius=0.04
- added link link_virtual_ft_sensor_lower, mass 0.04; collision cylinder length=0.025 radius=0.03; visual cylinder length=0.025 radius=0.03
- added link link_virtual_ft_sensor_upper, mass 0.05; collision cylinder length=0.0338 radius=0.034; visual cylinder length=0.0338 radius=0.034
- link left_inner_knuckle: geometry visual mesh filename=package://xarm_description/meshes/gripper/xarm/left_inner_k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
- link link1: geometry collision mesh filename=package://xarm_description/meshes/xarm7_1305/collision/link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; visual mesh filename=package://xarm_description/meshes/xarm7_1305/visual/link1.s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
- link link2: geometry collision mesh filename=package://xarm_description/meshes/xarm7_1305/collision/link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; visual mesh filename=package://xarm_description/meshes/xarm7_1305/visual/link2.s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
- link link3: geometry collision mesh filename=package://xarm_description/meshes/xarm7_1305/collision/link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; visual mesh filename=package://xarm_description/meshes/xarm7_1305/visual/link3.s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
- link link4: geometry collision mesh filename=package://xarm_description/meshes/xarm7_1305/collision/link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; visual mesh filename=package://xarm_description/meshes/xarm7_1305/visual/link4.s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
- link link5: geometry collision mesh filename=package://xarm_description/meshes/xarm7_1305/collision/link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; visual mesh filename=package://xarm_description/meshes/xarm7_1305/visual/link5.s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
- link link6: geometry collision mesh filename=package://xarm_description/meshes/xarm7_1305/collision/link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; visual mesh filename=package://xarm_description/meshes/xarm7_1305/visual/link6.s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
- link link7: geometry collision mesh filename=package://xarm_description/meshes/xarm7_1305/collision/link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; visual mesh filename=package://xarm_description/meshes/xarm7_1305/visual/link7.s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
- link link_base: geometry collision mesh filename=package://xarm_description/meshes/xarm7_1305/collision/link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; visual mesh filename=package://xarm_description/meshes/xarm7_1305/visual/link_ba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
- link right_inner_knuckle: geometry visual mesh filename=package://xarm_description/meshes/gripper/xarm/right_inner_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
Joints:
- added joint joint_tcp_ball: type fixed, parent link_tcp, child link_tcp_ball, origin xyz=0 0 0 rpy=0 0 0
- added joint joint_virtual_ft_sensor_lower: type fixed, parent link_virtual_ft_sensor_upper, child link_virtual_ft_sensor_lower, origin xyz=0 0 0.0294 rpy=0 0 0
- added joint joint_virtual_ft_sensor_upper: type fixed, parent link7, child link_virtual_ft_sensor_upper, origin xyz=0 0 0.0169 rpy=0 0 0
- joint joint_eef: origin xyz=0 0 0 rpy=0 0 0 -> xyz=0 0 0.0125 rpy=0 0 0; parent link7 -> link_virtual_ft_sensor_lower
