Commit message: refactor: move gripper collision boxes to base link

File: xarm7_1305_left_ball_ee_old.urdf (robot description, URDF)
Before this commit: robot UF_ROBOT, 31 links, 30 joints
Links:
- link left_outer_knuckle: geometry collision mesh filename=package://xarm_description/meshes/gripper/xarm/left_outer_k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; visual mesh filename=package://xarm_description/meshes/gripper/xarm/left_outer_k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
- link link_tcp_ball: mass 0.100 -> 0.00625; geometry collision sphere radius=0.03; visual sphere radius=0.02
- link right_outer_knuckle: geometry collision mesh filename=package://xarm_description/meshes/gripper/xarm/right_outer_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; visual mesh filename=package://xarm_description/meshes/gripper/xarm/right_outer_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
- link xarm_gripper_base_link: geometry collision mesh filename=package://xarm_description/meshes/gripper/xarm/base_link.stl; visual mesh filename=package://xarm_description/meshes/gripper/xarm/base_link.stl
Joints:
- joint drive_joint: limit lower=0.7310 upper=0.7310 effort=50 velocity=0 -> lower=0.7235 upper=0.7235 effort=50 velocity=0
- joint joint_tcp_stick: origin xyz=0 0 -0.00241 rpy=1.5707963267948966 0 1.5707963267948966 -> xyz=0 0 0.0315 rpy=1.5707963267948966 0 1.5707963267948966
- joint left_finger_joint: limit lower=0.7310 upper=0.7310 effort=50 velocity=0 -> lower=0.7235 upper=0.7235 effort=50 velocity=0
- joint left_inner_knuckle_joint: limit lower=0.7310 upper=0.7310 effort=50 velocity=0 -> lower=0.7235 upper=0.7235 effort=50 velocity=0
- joint right_finger_joint: limit lower=0.7310 upper=0.7310 effort=50 velocity=0 -> lower=0.7235 upper=0.7235 effort=50 velocity=0
- joint right_inner_knuckle_joint: limit lower=0.7310 upper=0.7310 effort=50 velocity=0 -> lower=0.7235 upper=0.7235 effort=50 velocity=0
- joint right_outer_knuckle_joint: limit lower=0.7310 upper=0.7310 effort=50 velocity=0 -> lower=0.7235 upper=0.7235 effort=50 velocity=0
