Commit message: feat: update dual xArm setup and URDFs

File: xarm7_1305_left_ball_ee.urdf (robot description, URDF)
Before this commit: robot UF_ROBOT, 30 links, 29 joints
Links:
- link left_outer_knuckle: geometry collision mesh filename=package://xarm_description/meshes/gripper/xarm/left_outer_k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; visual mesh filename=package://xarm_description/meshes/gripper/xarm/left_outer_k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
- link link1: mass 2.382 -> 2.507
- link link2: mass 1.869 -> 2.2812
- link link3: mass 1.6383 -> 2.0
- link link4: mass 1.7269 -> 2.1212
- link link5: mass 1.3203 -> 1.36
- link link6: mass 1.325 -> 1.345
- link link_tcp_ball: mass 0.05 -> 0.02109375; geometry collision sphere radius=0.03; visual sphere radius=0.03
- link right_outer_knuckle: geometry collision mesh filename=package://xarm_description/meshes/gripper/xarm/right_outer_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; visual mesh filename=package://xarm_description/meshes/gripper/xarm/right_outer_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
Joints:
- joint drive_joint: limit lower=0.55 upper=0.55 effort=50 velocity=0 -> lower=0 upper=0.85 effort=50 velocity=2
- joint left_finger_joint: limit lower=0.55 upper=0.55 effort=50 velocity=0 -> lower=0 upper=0.85 effort=50 velocity=2
- joint left_inner_knuckle_joint: limit lower=0.55 upper=0.55 effort=50 velocity=0 -> lower=0 upper=0.85 effort=50 velocity=2
- joint right_finger_joint: limit lower=0.55 upper=0.55 effort=50 velocity=0 -> lower=0 upper=0.85 effort=50 velocity=2
- joint right_inner_knuckle_joint: limit lower=0.55 upper=0.55 effort=50 velocity=0 -> lower=0 upper=0.85 effort=50 velocity=2
- joint right_outer_knuckle_joint: limit lower=0.55 upper=0.55 effort=50 velocity=0 -> lower=0 upper=0.85 effort=50 velocity=2

Commit message: feat: add dual xArm rollout and observation utilities

File: xarm7_1305_left_ball_ee.urdf (robot description, URDF)
Before this commit: robot UF_ROBOT, 30 links, 29 joints
Joints:
- joint drive_joint: limit lower=0 upper=0.85 effort=50 velocity=2 -> lower=0.55 upper=0.55 effort=50 velocity=0
- joint left_finger_joint: limit lower=0 upper=0.85 effort=50 velocity=2 -> lower=0.55 upper=0.55 effort=50 velocity=0
- joint left_inner_knuckle_joint: limit lower=0 upper=0.85 effort=50 velocity=2 -> lower=0.55 upper=0.55 effort=50 velocity=0
- joint right_finger_joint: limit lower=0 upper=0.85 effort=50 velocity=2 -> lower=0.55 upper=0.55 effort=50 velocity=0
- joint right_inner_knuckle_joint: limit lower=0 upper=0.85 effort=50 velocity=2 -> lower=0.55 upper=0.55 effort=50 velocity=0
- joint right_outer_knuckle_joint: limit lower=0 upper=0.85 effort=50 velocity=2 -> lower=0.55 upper=0.55 effort=50 velocity=0

Commit message: feat: add stick end effector and controller limits

File: xarm7_1305_left_ball_ee.urdf (robot description, URDF)
Before this commit: robot UF_ROBOT, 30 links, 29 joints
Links:
- added link link_tcp_stick, mass 0.05; collision mesh filename=xarm7_stick_centered.stl scale=0.001 0.001 0.001; visual mesh filename=xarm7_stick_centered.stl scale=0.001 0.001 0.001
- link link_tcp_ball: mass 0.02109375 -> 0.00625; geometry collision sphere radius=0.03; visual sphere radius=0.02
Joints:
- added joint joint_tcp_stick: type fixed, parent link_tcp, child link_tcp_stick, origin xyz=0 0 0 rpy=1.5707963267948966 0 1.5707963267948966
- joint joint_tcp_ball: origin xyz=0 0 0 rpy=0 0 0 -> xyz=0 0.0475 0 rpy=0 0 0; parent link_tcp -> link_tcp_stick

Commit message: feat: add gripper control and fix dual arm positioning

File: xarm7_1305_left_ball_ee.urdf (robot description, URDF)
Before this commit: robot UF_ROBOT, 31 links, 30 joints
Joints:
- joint joint_tcp_stick: origin xyz=0 0 0 rpy=1.5707963267948966 0 1.5707963267948966 -> xyz=0 0 0.0315 rpy=1.5707963267948966 0 1.5707963267948966

Commit message: feat: add joint trajectory visualization

File: xarm7_1305_left_ball_ee.urdf (robot description, URDF)
Before this commit: robot UF_ROBOT, 31 links, 30 joints
Joints:
- joint drive_joint: limit lower=0.55 upper=0.55 effort=50 velocity=0 -> lower=0.7235 upper=0.7235 effort=50 velocity=0
- joint left_finger_joint: limit lower=0.55 upper=0.55 effort=50 velocity=0 -> lower=0.7235 upper=0.7235 effort=50 velocity=0
- joint left_inner_knuckle_joint: limit lower=0.55 upper=0.55 effort=50 velocity=0 -> lower=0.7235 upper=0.7235 effort=50 velocity=0
- joint right_finger_joint: limit lower=0.55 upper=0.55 effort=50 velocity=0 -> lower=0.7235 upper=0.7235 effort=50 velocity=0
- joint right_inner_knuckle_joint: limit lower=0.55 upper=0.55 effort=50 velocity=0 -> lower=0.7235 upper=0.7235 effort=50 velocity=0
- joint right_outer_knuckle_joint: limit lower=0.55 upper=0.55 effort=50 velocity=0 -> lower=0.7235 upper=0.7235 effort=50 velocity=0

Commit message: tune: optimize robot control and scene parameters

File: xarm7_1305_left_ball_ee.urdf (robot description, URDF)
Before this commit: robot UF_ROBOT, 31 links, 30 joints
Links:
- link link_tcp_ball: mass 0.00625 -> 0.100
Joints:
- joint drive_joint: limit lower=0.7235 upper=0.7235 effort=50 velocity=0 -> lower=0.7310 upper=0.7310 effort=50 velocity=0
- joint joint_tcp_stick: origin xyz=0 0 0.0315 rpy=1.5707963267948966 0 1.5707963267948966 -> xyz=0 0 -0.00541 rpy=1.5707963267948966 0 1.5707963267948966
- joint left_finger_joint: limit lower=0.7235 upper=0.7235 effort=50 velocity=0 -> lower=0.7310 upper=0.7310 effort=50 velocity=0
- joint left_inner_knuckle_joint: limit lower=0.7235 upper=0.7235 effort=50 velocity=0 -> lower=0.7310 upper=0.7310 effort=50 velocity=0
- joint right_finger_joint: limit lower=0.7235 upper=0.7235 effort=50 velocity=0 -> lower=0.7310 upper=0.7310 effort=50 velocity=0
- joint right_inner_knuckle_joint: limit lower=0.7235 upper=0.7235 effort=50 velocity=0 -> lower=0.7310 upper=0.7310 effort=50 velocity=0
- joint right_outer_knuckle_joint: limit lower=0.7235 upper=0.7235 effort=50 velocity=0 -> lower=0.7310 upper=0.7310 effort=50 velocity=0

Commit message: refactor: update gripper collisions and box dimensions

File: xarm7_1305_left_ball_ee.urdf (robot description, URDF)
Before this commit: robot UF_ROBOT, 31 links, 30 joints
Links:
- link left_finger: geometry collision box size=0.03 0.08 0.0180; collision box size=0.032 0.01900 0.05693
- link left_outer_knuckle: geometry visual mesh filename=package://xarm_description/meshes/gripper/xarm/left_outer_k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
- link link_tcp_ball: geometry collision sphere radius=0.02; visual sphere radius=0.02
- link link_tcp_stick: geometry collision mesh filename=file:///home/jika/Desktop/my_projects/robot/maniskill_exp/x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 scale=0.001 0.001 0.001; visual mesh filename=file:///home/jika/Desktop/my_projects/robot/maniskill_exp/x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 scale=0.001 0.001 0.001
- link right_finger: geometry collision box size=0.03 0.08 0.0180; collision box size=0.032 0.01900 0.05693
- link right_outer_knuckle: geometry visual mesh filename=package://xarm_description/meshes/gripper/xarm/right_outer_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
- link xarm_gripper_base_link: geometry collision box size=0.075 0.1222 0.0900; visual mesh filename=package://xarm_description/meshes/gripper/xarm/base_link.stl
Joints:
- joint joint_tcp_stick: origin xyz=0 0 -0.00541 rpy=1.5707963267948966 0 1.5707963267948966 -> xyz=0 0 -0.00241 rpy=1.5707963267948966 0 1.5707963267948966

Commit message: feat: optimize contact handling and reward structure

File: xarm7_1305_left_ball_ee.urdf (robot description, URDF)
Before this commit: robot UF_ROBOT, 31 links, 30 joints
Links:
- link link1: geometry collision mesh filename=package://xarm_description/meshes/xarm7_1305/collision/link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 scale=1.20 1.20 1.20; visual mesh filename=package://xarm_description/meshes/xarm7_1305/visual/link1.s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 scale=1.20 1.20 1.20
- link link2: geometry collision mesh filename=package://xarm_description/meshes/xarm7_1305/collision/link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 scale=1.20 1.20 1.20; visual mesh filename=package://xarm_description/meshes/xarm7_1305/visual/link2.s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 scale=1.20 1.20 1.20
- link xarm_gripper_base_link: geometry collision box size=0.03 0.06 0.024; collision box size=0.03 0.06 0.024

Commit message: feat: add box pose assets and tune xArm contact settings

File: xarm7_1305_left_ball_ee.urdf (robot description, URDF)
Before this commit: robot UF_ROBOT, 31 links, 30 joints
Links:
- link link_virtual_ft_sensor_lower: geometry collision cylinder length=0.025 radius=0.035; visual cylinder length=0.025 radius=0.035
- link link_virtual_ft_sensor_upper: geometry collision cylinder length=0.0338 radius=0.035; visual cylinder length=0.0338 radius=0.035
