Commit message: feat: add force-sensor-free xarm ball ee agent

File: xarm7_1305_left_ball_ee_wo_force_sensor.urdf (robot description, URDF)
Before this commit: robot UF_ROBOT, 31 links, 30 joints
Links:
- removed link link_virtual_ft_sensor_lower
- removed link link_virtual_ft_sensor_upper
Joints:
- removed joint joint_virtual_ft_sensor_lower
- removed joint joint_virtual_ft_sensor_upper
- joint joint_eef: origin xyz=0 0 0.0125 rpy=0 0 0 -> xyz=0 0 0 rpy=0 0 0; parent link_virtual_ft_sensor_lower -> link7
