Commit message: fix(urdf): narrow xArm joint7 limits

File: robotagents/xarm7_wo_gripper.urdf (robot description, URDF)
Before this commit: robot UF_ROBOT_XARM7_NO_GRIPPER, 10 links, 9 joints
Joints:
- joint joint6: limit lower=-1.69297 upper=3.141592653589793 effort=20 velocity=3.14 -> lower=-1.5707963267948966 upper=1.5707963267948966 effort=20 velocity=3.14

File: xarm7.urdf (robot description, URDF)
Before this commit: robot UF_ROBOT, 18 links, 17 joints
Joints:
- joint joint6: limit lower=-1.69297 upper=3.141592653589793 effort=20 velocity=3.14 -> lower=-1.5707963267948966 upper=1.5707963267948966 effort=20 velocity=3.14
