Commit message: chore: simplify xarm7 visualization urdf

File: robotagents/assets/xarm7/xarm7_1305_left.urdf (robot description, URDF)
Before this commit: robot UF_ROBOT, 27 links, 26 joints
Links:
- link left_finger: geometry visual mesh filename=package://xarm_description/meshes/gripper/xarm/left_finger.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
- link left_inner_knuckle: geometry visual mesh filename=package://xarm_description/meshes/gripper/xarm/left_inner_k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
- link left_outer_knuckle: geometry visual mesh filename=package://xarm_description/meshes/gripper/xarm/left_outer_k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
- link link_eef: geometry visual mesh filename=package://xarm_description/meshes/camera/realsense/visual/d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
- link right_finger: geometry visual mesh filename=package://xarm_description/meshes/gripper/xarm/right_finger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
- link right_inner_knuckle: geometry visual mesh filename=package://xarm_description/meshes/gripper/xarm/right_inner_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
- link right_outer_knuckle: geometry visual mesh filename=package://xarm_description/meshes/gripper/xarm/right_outer_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
- link xarm_gripper_base_link: geometry visual mesh filename=package://xarm_description/meshes/gripper/xarm/base_link.stl

Commit message: chore: add rviz panda visualization urdf

File: robotagents/assets/xarm7/xarm7_1305_left.urdf (robot description, URDF)
Before this commit: robot UF_ROBOT, 27 links, 26 joints
Links:
- link left_finger: geometry collision box size=0.028 0.010 0.036; visual mesh filename=package://xarm_description/meshes/gripper/xarm/left_finger.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
- link right_finger: geometry collision box size=0.028 0.010 0.036; visual mesh filename=package://xarm_description/meshes/gripper/xarm/right_finger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

Commit message: chore: update xarm7 finger collision mesh

File: robotagents/assets/xarm7/xarm7_1305_left.urdf (robot description, URDF)
Before this commit: robot UF_ROBOT, 27 links, 26 joints
Links:
- link left_finger: geometry collision mesh filename=package://xarm_description/meshes/gripper/xarm/left_finger.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; visual mesh filename=package://xarm_description/meshes/gripper/xarm/left_finger.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
- link right_finger: geometry collision mesh filename=package://xarm_description/meshes/gripper/xarm/right_finger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; visual mesh filename=package://xarm_description/meshes/gripper/xarm/right_finger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

Commit message: changed the finger collision mesh

File: robotagents/assets/xarm7/xarm7_1305_left.urdf (robot description, URDF)
Before this commit: robot UF_ROBOT, 27 links, 26 joints
Links:
- link left_finger: geometry visual mesh filename=package://xarm_description/meshes/gripper/xarm/left_finger.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
- link right_finger: geometry visual mesh filename=package://xarm_description/meshes/gripper/xarm/right_finger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

Commit message: feat: add repaired xarm finger meshes

File: robotagents/assets/xarm7/xarm7_1305_left.urdf (robot description, URDF)
Before this commit: robot UF_ROBOT, 27 links, 26 joints
Links:
- link left_finger: geometry collision box size=0.028 0.010 0.036; visual mesh filename=file:///home/kotaro/my_projects/robotics/maniskill_exp/xarm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 scale=0.001 0.001 0.001
- link right_finger: geometry collision box size=0.028 0.010 0.036; visual mesh filename=file:///home/kotaro/my_projects/robotics/maniskill_exp/xarm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 scale=0.001 0.001 0.001

Commit message: fix: use relative xarm finger mesh paths

File: robotagents/assets/xarm7/xarm7_1305_left.urdf (robot description, URDF)
Before this commit: robot UF_ROBOT, 27 links, 26 joints
Links:
- link left_finger: geometry collision box size=0.028 0.010 0.036; visual mesh filename=../../../xarm_description/meshes/gripper/xarm/left_kirisute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 scale=0.001 0.001 0.001
- link right_finger: geometry collision box size=0.028 0.010 0.036; visual mesh filename=../../../xarm_description/meshes/gripper/xarm/right_kirisut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 scale=0.001 0.001 0.001

Commit message: fix: use kirisute meshes for finger collisions

File: robotagents/assets/xarm7/xarm7_1305_left.urdf (robot description, URDF)
Before this commit: robot UF_ROBOT, 27 links, 26 joints
Links:
- link left_finger: geometry collision mesh filename=../../../xarm_description/meshes/gripper/xarm/left_kirisute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 scale=0.001 0.001 0.001; visual mesh filename=../../../xarm_description/meshes/gripper/xarm/left_kirisute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 scale=0.001 0.001 0.001
- link right_finger: geometry collision mesh filename=../../../xarm_description/meshes/gripper/xarm/right_kirisut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 scale=0.001 0.001 0.001; visual mesh filename=../../../xarm_description/meshes/gripper/xarm/right_kirisut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 scale=0.001 0.001 0.001

Commit message: feat: visualize left finger tip marker

File: robotagents/assets/xarm7/xarm7_1305_left.urdf (robot description, URDF)
Before this commit: robot UF_ROBOT, 27 links, 26 joints
Links:
- link left_finger: geometry collision mesh filename=../../../xarm_description/meshes/gripper/xarm/left_kirisute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 scale=0.001 0.001 0.001; visual mesh filename=../../../xarm_description/meshes/gripper/xarm/left_kirisute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 scale=0.001 0.001 0.001

Commit message: fix: test xarm gripper mimic with nightly

File: robotagents/assets/xarm7/xarm7_1305_left.urdf (robot description, URDF)
Before this commit: robot UF_ROBOT, 27 links, 26 joints
Links:
- link left_finger: geometry collision box size=0.012 0.006 0.040; visual box size=0.012 0.006 0.040
- link right_finger: geometry collision box size=0.012 0.006 0.040; visual box size=0.012 0.006 0.040
Joints:
- removed joint drive_joint
- removed joint right_outer_knuckle_joint
- added joint left_drive_joint: type revolute, parent xarm_gripper_base_link, child left_outer_knuckle, origin xyz=0 0.035 0.059098 rpy=0 0 0, axis 1 0 0, limit lower=0 upper=0.85 effort=50 velocity=2
- added joint right_drive_joint: type revolute, parent xarm_gripper_base_link, child right_outer_knuckle, origin xyz=0 -0.035 0.059098 rpy=0 0 0, axis -1 0 0, limit lower=0 upper=0.85 effort=50 velocity=2
- joint left_finger_joint: mimic joint=drive_joint multiplier=1 offset=0 -> joint=left_drive_joint multiplier=1 offset=0
- joint left_inner_knuckle_joint: mimic joint=drive_joint multiplier=1 offset=0 -> joint=left_drive_joint multiplier=1 offset=0
- joint right_finger_joint: mimic joint=drive_joint multiplier=1 offset=0 -> joint=right_drive_joint multiplier=1 offset=0
- joint right_inner_knuckle_joint: mimic joint=drive_joint multiplier=1 offset=0 -> joint=right_drive_joint multiplier=1 offset=0

Commit message: feat: tune cardboard drawer open reward

File: robotagents/assets/xarm7/xarm7_1305_left.urdf (robot description, URDF)
Before this commit: robot UF_ROBOT, 27 links, 26 joints
Links:
- link left_outer_knuckle: geometry collision mesh filename=package://xarm_description/meshes/gripper/xarm/left_outer_k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; visual mesh filename=package://xarm_description/meshes/gripper/xarm/left_outer_k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
- link right_outer_knuckle: geometry collision mesh filename=package://xarm_description/meshes/gripper/xarm/right_outer_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; visual mesh filename=package://xarm_description/meshes/gripper/xarm/right_outer_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
- link xarm_gripper_base_link: geometry collision mesh filename=package://xarm_description/meshes/gripper/xarm/base_link.stl; visual mesh filename=package://xarm_description/meshes/gripper/xarm/base_link.stl

Commit message: fix: restore box xarm finger geometry

File: robotagents/assets/xarm7/xarm7_1305_left.urdf (robot description, URDF)
Before this commit: robot UF_ROBOT, 27 links, 26 joints
Links:
- link left_finger: geometry collision box size=0.012 0.006 0.040; visual box size=0.012 0.006 0.040
- link right_finger: geometry collision box size=0.012 0.006 0.040; visual box size=0.012 0.006 0.040

Commit message: fix: use box finger collisions

File: robotagents/assets/xarm7/xarm7_1305_left.urdf (robot description, URDF)
Before this commit: robot UF_ROBOT, 27 links, 26 joints
Links:
- link left_finger: geometry collision box size=0.012 0.006 0.040; collision box size=0.012 0.01 0.010
- link right_finger: geometry collision box size=0.012 0.006 0.040; collision box size=0.012 0.01 0.010
