Commit message: fix: update kinematics gripper urdf joints

File: robotagents/assets/xarm7/xarm7_1305_gripper_realsense_sn_kinematics.urdf (robot description, URDF)
Before this commit: robot UF_ROBOT, 27 links, 26 joints
Links:
- link left_inner_knuckle: geometry visual mesh filename=package://xarm_description/meshes/gripper/xarm/left_inner_k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
- link right_inner_knuckle: geometry visual mesh filename=package://xarm_description/meshes/gripper/xarm/right_inner_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
Joints:
- removed joint drive_joint
- removed joint right_outer_knuckle_joint
- added joint left_drive_joint: type revolute, parent xarm_gripper_base_link, child left_outer_knuckle, origin xyz=0 0.035 0.059098 rpy=0 0 0, axis 1 0 0, limit lower=0 upper=0.85 effort=500 velocity=2
- added joint right_drive_joint: type revolute, parent xarm_gripper_base_link, child right_outer_knuckle, origin xyz=0 -0.035 0.059098 rpy=0 0 0, axis -1 0 0, limit lower=0 upper=0.85 effort=500 velocity=2
- joint left_finger_joint: limit lower=0 upper=0.85 effort=50 velocity=2 -> lower=0 upper=0.85 effort=500 velocity=2; mimic joint=drive_joint multiplier=1 offset=0 -> joint=left_drive_joint multiplier=1 offset=0
- joint left_inner_knuckle_joint: limit lower=0 upper=0.85 effort=50 velocity=2 -> lower=0 upper=0.85 effort=500 velocity=2; mimic joint=drive_joint multiplier=1 offset=0 -> joint=left_drive_joint multiplier=1 offset=0
- joint right_finger_joint: limit lower=0 upper=0.85 effort=50 velocity=2 -> lower=0 upper=0.85 effort=500 velocity=2; mimic joint=drive_joint multiplier=1 offset=0 -> joint=right_drive_joint multiplier=1 offset=0
- joint right_inner_knuckle_joint: limit lower=0 upper=0.85 effort=50 velocity=2 -> lower=0 upper=0.85 effort=500 velocity=2; mimic joint=drive_joint multiplier=1 offset=0 -> joint=right_drive_joint multiplier=1 offset=0

Commit message: fix: use nominal xarm urdf in legacy agent

File: robotagents/assets/xarm7/xarm7_1305_gripper_realsense_sn_kinematics.urdf (robot description, URDF)
Before this commit: robot UF_ROBOT, 27 links, 26 joints
Links:
- link link_eef: geometry visual mesh filename=package://xarm_description/meshes/camera/realsense/visual/d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

Commit message: fix: widen xarm finger collision boxes

File: robotagents/assets/xarm7/xarm7_1305_gripper_realsense_sn_kinematics.urdf (robot description, URDF)
Before this commit: robot UF_ROBOT, 27 links, 26 joints
Links:
- link left_finger: geometry collision box size=0.012 0.0075 0.040; collision box size=0.012 0.01 0.010
- link right_finger: geometry collision box size=0.012 0.0075 0.040; collision box size=0.012 0.01 0.010

File: robotagents/assets/xarm7/xarm7_1305_left.urdf (robot description, URDF)
Before this commit: robot UF_ROBOT, 27 links, 26 joints
Links:
- link left_finger: geometry collision box size=0.012 0.0075 0.040; collision box size=0.012 0.01 0.010
- link right_finger: geometry collision box size=0.012 0.0075 0.040; collision box size=0.012 0.01 0.010

Commit message: fix: limit raised cardboard variant to randomized envs

File: robotagents/assets/xarm7/xarm7_1305_gripper_realsense_sn_kinematics.urdf (robot description, URDF)
Before this commit: robot UF_ROBOT, 27 links, 26 joints
Links:
- link left_finger: geometry collision box size=0.012 0.006 0.040; collision box size=0.012 0.01 0.010
- link right_finger: geometry collision box size=0.012 0.006 0.040; collision box size=0.012 0.01 0.010

File: robotagents/assets/xarm7/xarm7_1305_left.urdf (robot description, URDF)
Before this commit: robot UF_ROBOT, 27 links, 26 joints
Links:
- link left_finger: geometry collision box size=0.012 0.006 0.040; collision box size=0.012 0.01 0.010
- link right_finger: geometry collision box size=0.012 0.006 0.040; collision box size=0.012 0.01 0.010
