Commit message: refactor: organize xarm kinematics urdfs

File: robotagents/assets/xarm7/xarm7_1305_left_ball_ee_wo_force_sensor_kinematics.urdf (robot description, URDF)
Before this commit: robot UF_ROBOT, 31 links, 30 joints
Links:
- removed link link_virtual_ft_sensor_lower
- removed link link_virtual_ft_sensor_upper
- link left_outer_knuckle: geometry visual mesh filename=package://xarm_description/meshes/gripper/xarm/left_outer_k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
- link link1: geometry collision mesh filename=package://xarm_description/meshes/xarm7_1305/collision/link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 scale=1.20 1.20 1.20; visual mesh filename=package://xarm_description/meshes/xarm7_1305/visual/link1.s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 scale=1.20 1.20 1.20
- link link2: geometry collision mesh filename=package://xarm_description/meshes/xarm7_1305/collision/link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 scale=1.20 1.20 1.20; visual mesh filename=package://xarm_description/meshes/xarm7_1305/visual/link2.s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 scale=1.20 1.20 1.20
- link link_tcp_ball: mass 0.00625 -> 0.100; geometry collision sphere radius=0.02; visual sphere radius=0.02
- link link_tcp_stick: geometry collision mesh filename=../../../xarm7_stick_centered.stl scale=0.001 0.001 0.001; visual mesh filename=../../../xarm7_stick_centered.stl scale=0.001 0.001 0.001
- link right_outer_knuckle: geometry visual mesh filename=package://xarm_description/meshes/gripper/xarm/right_outer_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
- link xarm_gripper_base_link: geometry collision box size=0.03 0.06 0.024; collision box size=0.03 0.06 0.024
Joints:
- removed joint joint_virtual_ft_sensor_lower
- removed joint joint_virtual_ft_sensor_upper
- joint drive_joint: limit lower=0.7235 upper=0.7235 effort=50 velocity=0 -> lower=0.7310 upper=0.7310 effort=50 velocity=0
- joint joint1: origin xyz=0 0 0.267 rpy=0 0 0 -> xyz=-0.0013510942226275802 0.00013545599358621985 0.2658418118953705 rpy=-0.0013863248750567436 -0.0026416119653731585 1.8310676068722387e-06
- joint joint2: origin xyz=0 0 0 rpy=-1.5708 0 0 -> xyz=0.0004150629392825067 -0.00019739395065698773 3.5883675764125655e-07 rpy=-1.5726187229156494 0.0026415116153657436 -0.00045838893856853247
- joint joint3: origin xyz=0 -0.293 0 rpy=1.5708 0 0 -> xyz=0.00013824999041389674 -0.29250088334083557 -0.0009382066200487316 rpy=1.57400381565094 -0.0004602178232744336 -7.380804731837998e-07
- joint joint4: origin xyz=0.0525 0 0 rpy=1.5708 0 0 -> xyz=0.05247224494814873 0.0012199928751215339 6.521167051687371e-06 rpy=1.5755400657653809 7.002831807767507e-06 -0.0029524490237236023
- joint joint5: origin xyz=0.0775 -0.3425 0 rpy=1.5708 0 0 -> xyz=0.07674738764762878 -0.3424482047557831 0.0021595987491309643 rpy=1.5644944906234741 0.0029679781291633844 0.0028048199601471424
- joint joint6: origin xyz=0 0 0 rpy=1.5708 0 0 -> xyz=0.0005820331862196326 -0.0029558769892901182 -5.6971024605445564e-05 rpy=1.5900721549987793 -0.0027992529794573784 -0.0012112014228478074
- joint joint7: origin xyz=0.076 0.097 0 rpy=-1.5708 0 0 -> xyz=0.07630979269742966 0.09632150083780289 -0.0017321980558335781 rpy=-1.5888656377792358 0.0008275225991383195 -0.00014797094627283514
- joint joint_eef: origin xyz=0 0 0.0125 rpy=0 0 0 -> xyz=0 0 0 rpy=0 0 0; parent link_virtual_ft_sensor_lower -> link7
- joint joint_tcp_stick: origin xyz=0 0 0.0315 rpy=1.5707963267948966 0 1.5707963267948966 -> xyz=0 0 -0.00241 rpy=1.5707963267948966 0 1.5707963267948966
- joint left_finger_joint: limit lower=0.7235 upper=0.7235 effort=50 velocity=0 -> lower=0.7310 upper=0.7310 effort=50 velocity=0
- joint left_inner_knuckle_joint: limit lower=0.7235 upper=0.7235 effort=50 velocity=0 -> lower=0.7310 upper=0.7310 effort=50 velocity=0
- joint right_finger_joint: limit lower=0.7235 upper=0.7235 effort=50 velocity=0 -> lower=0.7310 upper=0.7310 effort=50 velocity=0
- joint right_inner_knuckle_joint: limit lower=0.7235 upper=0.7235 effort=50 velocity=0 -> lower=0.7310 upper=0.7310 effort=50 velocity=0
- joint right_outer_knuckle_joint: limit lower=0.7235 upper=0.7235 effort=50 velocity=0 -> lower=0.7310 upper=0.7310 effort=50 velocity=0

File: robotagents/assets/xarm7/xarm7_1305_right_ball_ee_wo_force_sensor_kinematics.urdf (robot description, URDF)
Before this commit: robot UF_ROBOT, 18 links, 17 joints
Links:
- added link camera_color_frame
- added link camera_color_optical_frame
- added link camera_depth_frame
- added link camera_depth_optical_frame
- added link camera_left_ir_frame
- added link camera_left_ir_optical_frame
- added link camera_link
- added link camera_right_ir_frame
- added link camera_right_ir_optical_frame
- added link link_tcp_ball, mass 0.100; collision sphere radius=0.02; visual sphere radius=0.02
- added link link_tcp_stick, mass 0.05; collision mesh filename=../../../xarm7_stick_centered.stl scale=0.001 0.001 0.001; visual mesh filename=../../../xarm7_stick_centered.stl scale=0.001 0.001 0.001
- link left_finger: geometry visual mesh filename=package://xarm_description/meshes/gripper/xarm/left_finger.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
- link left_inner_knuckle: geometry visual mesh filename=package://xarm_description/meshes/gripper/xarm/left_inner_k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
- link left_outer_knuckle: geometry visual mesh filename=package://xarm_description/meshes/gripper/xarm/left_outer_k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
- link link1: mass 2.382 -> 2.507; geometry collision mesh filename=package://xarm_description/meshes/xarm7_1305/collision/link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 scale=1.20 1.20 1.20; visual mesh filename=package://xarm_description/meshes/xarm7_1305/visual/link1.s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 scale=1.20 1.20 1.20
- link link2: mass 1.869 -> 2.2812; geometry collision mesh filename=package://xarm_description/meshes/xarm7_1305/collision/link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 scale=1.20 1.20 1.20; visual mesh filename=package://xarm_description/meshes/xarm7_1305/visual/link2.s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 scale=1.20 1.20 1.20
- link link3: mass 1.6383 -> 2.0; geometry collision mesh filename=package://xarm_description/meshes/xarm7_1305/collision/link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; visual mesh filename=package://xarm_description/meshes/xarm7_1305/visual/link3.s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
- link link4: mass 1.7269 -> 2.1212; geometry collision mesh filename=package://xarm_description/meshes/xarm7_1305/collision/link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; visual mesh filename=package://xarm_description/meshes/xarm7_1305/visual/link4.s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
- link link5: mass 1.3203 -> 1.36; geometry collision mesh filename=package://xarm_description/meshes/xarm7_1305/collision/link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; visual mesh filename=package://xarm_description/meshes/xarm7_1305/visual/link5.s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
- link link6: mass 1.325 -> 1.345; geometry collision mesh filename=package://xarm_description/meshes/xarm7_1305/collision/link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; visual mesh filename=package://xarm_description/meshes/xarm7_1305/visual/link6.s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
- link link7: geometry collision mesh filename=package://xarm_description/meshes/xarm7_1305/collision/link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; visual mesh filename=package://xarm_description/meshes/xarm7_1305/visual/link7.s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
- link link_base: geometry collision mesh filename=package://xarm_description/meshes/xarm7_1305/collision/link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; visual mesh filename=package://xarm_description/meshes/xarm7_1305/visual/link_ba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
- link link_eef: geometry collision mesh filename=package://xarm_description/meshes/camera/realsense/collisio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; visual mesh filename=package://xarm_description/meshes/camera/realsense/visual/d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
- link right_finger: geometry visual mesh filename=package://xarm_description/meshes/gripper/xarm/right_finger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
- link right_inner_knuckle: geometry visual mesh filename=package://xarm_description/meshes/gripper/xarm/right_inner_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
- link right_outer_knuckle: geometry visual mesh filename=package://xarm_description/meshes/gripper/xarm/right_outer_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
- link xarm_gripper_base_link: geometry collision box size=0.03 0.06 0.024; collision box size=0.03 0.06 0.024
Joints:
- added joint camera_color_joint: type fixed, parent camera_link, child camera_color_frame, origin xyz=0 0.015 0 rpy=0 0 0
- added joint camera_color_optical_joint: type fixed, parent camera_color_frame, child camera_color_optical_frame, origin xyz=0 0 0 rpy=-1.5707963267948966 0 -1.5707963267948966
- added joint camera_depth_joint: type fixed, parent camera_link, child camera_depth_frame, origin xyz=0 0 0 rpy=0 0 0
- added joint camera_depth_optical_joint: type fixed, parent camera_depth_frame, child camera_depth_optical_frame, origin xyz=0 0 0 rpy=-1.5707963267948966 0 -1.5707963267948966
- added joint camera_left_ir_joint: type fixed, parent camera_link, child camera_left_ir_frame, origin xyz=0 0 0 rpy=0 0 0
- added joint camera_left_ir_optical_joint: type fixed, parent camera_left_ir_frame, child camera_left_ir_optical_frame, origin xyz=0 0 0 rpy=-1.5707963267948966 0 -1.5707963267948966
- added joint camera_link_joint: type fixed, parent link_eef, child camera_link, origin xyz=0.06746 -0.0175 0.0237 rpy=3.141592653589793 -1.5707963267948966 0
- added joint camera_right_ir_joint: type fixed, parent camera_link, child camera_right_ir_frame, origin xyz=0 -0.050 0 rpy=0 0 0
- added joint camera_right_ir_optical_joint: type fixed, parent camera_right_ir_frame, child camera_right_ir_optical_frame, origin xyz=0 0 0 rpy=-1.5707963267948966 0 -1.5707963267948966
- added joint joint_tcp_ball: type fixed, parent link_tcp_stick, child link_tcp_ball, origin xyz=0 0.0475 0 rpy=0 0 0
- added joint joint_tcp_stick: type fixed, parent link_tcp, child link_tcp_stick, origin xyz=0 0 -0.00241 rpy=1.5707963267948966 0 1.5707963267948966
- joint drive_joint: limit lower=0 upper=0.85 effort=50 velocity=2 -> lower=0.7310 upper=0.7310 effort=50 velocity=0
- joint joint1: origin xyz=0 0 0.267 rpy=0 0 0 -> xyz=-0.0013503426453098655 0.00018677444313652813 0.26539966464042664 rpy=-0.0010736589320003986 -0.002312414813786745 1.2413730701155146e-06
- joint joint2: origin xyz=0 0 0 rpy=-1.5708 0 0 -> xyz=5.8161642613185904e-08 -0.00034268395393155515 -6.091162276788964e-07 rpy=-1.5690196752548218 0.0023149799089878798 -0.0017987253377214074
- joint joint3: origin xyz=0 -0.293 0 rpy=1.5708 0 0 -> xyz=0.00028617726638913155 -0.29286816716194153 -0.001043715630657971 rpy=1.5743601322174072 -0.0017984152073040605 -0.0010833805426955223
- joint joint4: origin xyz=0.0525 0 0 rpy=1.5708 0 0 -> xyz=0.0528821125626564 0.0009186743991449475 2.2439674012275646e-06 rpy=1.572906494140625 0.001081056077964604 -0.0027423850260674953
- joint joint5: origin xyz=0.0775 -0.3425 0 rpy=1.5708 0 0 -> xyz=0.07610870152711868 -0.3421746790409088 0.0011450782185420394 rpy=1.5674524307250977 0.0027586470823735 0.0038138972595334053
- joint joint6: origin xyz=0 0 0 rpy=1.5708 0 0 -> xyz=0.0006870674551464617 -0.003908557817339897 -7.96470048953779e-05 rpy=1.591173529624939 -0.0038158921524882317 -0.0007752391393296421
- joint joint7: origin xyz=0.076 0.097 0 rpy=-1.5708 0 0 -> xyz=0.07676228135824203 0.09626951068639755 -0.0021900306455790997 rpy=-1.5947095155715942 0.0003195755125489086 -0.00023540361144114286
- joint left_finger_joint: limit lower=0 upper=0.85 effort=50 velocity=2 -> lower=0.7310 upper=0.7310 effort=50 velocity=0
- joint left_inner_knuckle_joint: limit lower=0 upper=0.85 effort=50 velocity=2 -> lower=0.7310 upper=0.7310 effort=50 velocity=0
- joint right_finger_joint: limit lower=0 upper=0.85 effort=50 velocity=2 -> lower=0.7310 upper=0.7310 effort=50 velocity=0
- joint right_inner_knuckle_joint: limit lower=0 upper=0.85 effort=50 velocity=2 -> lower=0.7310 upper=0.7310 effort=50 velocity=0
- joint right_outer_knuckle_joint: limit lower=0 upper=0.85 effort=50 velocity=2 -> lower=0.7310 upper=0.7310 effort=50 velocity=0
